Commit message: added first arm link and second joint

File: urdf/robot.urdf (robot description, URDF)
Before this commit: robot mearm, 3 links, 2 joints
Links:
- removed link joint_0_link
- added link arm_0; collision mesh filename=package://mearm_model/meshes/arm_0_base.stl scale=0.001 0.001 0.001; collision mesh filename=package://mearm_model/meshes/arm_0_left.stl scale=0.001 0.001 0.001
- added link column; collision mesh filename=package://mearm_model/meshes/column_base.stl scale=0.001 0.001 0.001; collision mesh filename=package://mearm_model/meshes/column_board.stl scale=0.001 0.001 0.001
- link base_link: geometry collision mesh filename=package://mearm_model/meshes/base.stl scale=0.001 0.001 0.001; collision mesh filename=package://mearm_model/meshes/base_top.stl scale=0.001 0.001 0.001
Joints:
- added joint joint_1: type revolute, parent column, child arm_0, origin xyz=0.014 0 0.029 rpy=1.5707 -1.5707 0, axis 0 0 1, limit lower=-1.57 upper=1.0 effort=1000.0 velocity=0.5
- joint joint_0: child joint_0_link -> column

Commit message: added second part of arm

File: urdf/robot.urdf (robot description, URDF)
Before this commit: robot mearm, 4 links, 3 joints
Links:
- added link arm_1; visual mesh filename=package://mearm_model/meshes/arm_1_connector.stl scale=0.001 0.001 0.001; visual mesh filename=package://mearm_model/meshes/arm_1_left.stl scale=0.001 0.001 0.001
Joints:
- added joint joint_2: type revolute, parent arm_0, child arm_1, origin xyz=0.08 0 0, axis 0 0 1, limit lower=-1.57 upper=0.0 effort=1000.0 velocity=0.5

Commit message: added arm_1 servo actuator

File: urdf/robot.urdf (robot description, URDF)
Before this commit: robot mearm, 5 links, 4 joints
Links:
- added link arm_1_actuator; visual mesh filename=package://mearm_model/meshes/servo_actuator.stl scale=0.001 0.001 0.001
Joints:
- added joint joint_x: type revolute, parent column, child arm_1_actuator, origin xyz=0.015 0.01 0.03 rpy=1.57 0 3.14, axis 0 0 1, limit lower=0.0 upper=1.57 effort=1000.0 velocity=0.5, mimic joint=joint_2 multiplier=-1 offset=0
- joint joint_2: limit lower=-1.57 upper=0.0 effort=1000.0 velocity=0.5 -> lower=-1.57 upper=0.4 effort=1000.0 velocity=0.5

Commit message: properly moving connector

File: urdf/robot.urdf (robot description, URDF)
Before this commit: robot mearm, 6 links, 5 joints
Links:
- added link arm_0_1_connector; visual mesh filename=package://mearm_model/meshes/arm_1_connector.stl scale=0.001 0.001 0.001
- added link arm_0_support; visual mesh filename=package://mearm_model/meshes/arm_1_right.stl scale=0.001 0.001 0.001
- link arm_1: geometry visual mesh filename=package://mearm_model/meshes/arm_1_left.stl scale=0.001 0.001 0.001; visual mesh filename=package://mearm_model/meshes/arm_1_right.stl scale=0.001 0.001 0.001
Joints:
- added joint arm_0_connector_mimic: type revolute, parent arm_0, child arm_0_1_connector, origin xyz=0.08 0 0, axis 0 0 1, limit lower=-1.57 upper=1.57 effort=1000.0 velocity=0.5, mimic joint=joint_1 multiplier=-1 offset=-1.57
- added joint arm_0_support_mimic: type revolute, parent column, child arm_0_support, origin xyz=-0.021 -0.019 0.045 rpy=1.57 0 0, axis 0 0 1, limit lower=0.0 upper=1.57 effort=1000.0 velocity=0.5, mimic joint=joint_1 multiplier=1 offset=1.57

Commit message: added support for arm_1 link

File: urdf/robot.urdf (robot description, URDF)
Before this commit: robot mearm, 8 links, 7 joints
Links:
- removed link arm_1_actuator
- added link arm_1_actuator_0; visual mesh filename=package://mearm_model/meshes/servo_actuator.stl scale=0.001 0.001 0.001
- added link arm_1_actuator_1; visual mesh filename=package://mearm_model/meshes/arm_1_right.stl scale=0.001 0.001 0.001
- link arm_1: geometry visual mesh filename=package://mearm_model/meshes/arm_1_left.stl scale=0.001 0.001 0.001; visual mesh filename=package://mearm_model/meshes/arm_1_right.stl scale=0.001 0.001 0.001
Joints:
- removed joint joint_x
- added joint joint_2_mimic_0: type revolute, parent arm_1_actuator_0, child arm_1_actuator_1, origin xyz=0.035 0 0, axis 0 0 1, limit lower=-1.57 upper=0.4 effort=1000.0 velocity=0.5, mimic joint=joint_2 multiplier=-1 offset=1.57
- added joint joint_2_mimic_1: type revolute, parent arm_0, child arm_1, origin xyz=0.08 0 0, axis 0 0 1, limit lower=-1.57 upper=0.4 effort=1000.0 velocity=0.5, mimic joint=joint_2 multiplier=-1 offset=-1.57
- joint joint_2: child arm_1 -> arm_1_actuator_0; limit lower=-1.57 upper=0.4 effort=1000.0 velocity=0.5 -> lower=0.0 upper=1.57 effort=1000.0 velocity=0.5; origin xyz=0.08 0 0 -> xyz=0.015 0.01 0.03 rpy=1.57 0 3.14; parent arm_0 -> column

Commit message: added support for arm_1 link

File: urdf/robot.urdf (robot description, URDF)
Before this commit: robot mearm, 9 links, 8 joints
Links:
- added link arm_1_support; visual mesh filename=package://mearm_model/meshes/arm_1_right.stl scale=0.001 0.001 0.001
- link arm_1: geometry visual mesh filename=package://mearm_model/meshes/arm_1_left.stl scale=0.001 0.001 0.001; visual mesh filename=package://mearm_model/meshes/arm_1_right.stl scale=0.001 0.001 0.001
Joints:
- added joint arm_1_support_mimic: type revolute, parent arm_0_1_connector, child arm_1_support, origin xyz=0.012 0.018 0.014 rpy=0 0 1.57, axis 0 0 1, limit lower=-1.57 upper=0.4 effort=1000.0 velocity=0.5, mimic joint=joint_2 multiplier=-1 offset=-1.57

Commit message: added virtual link to mimic multiple joints in arm1 support

File: urdf/robot.urdf (robot description, URDF)
Before this commit: robot mearm, 10 links, 9 joints
Links:
- removed link arm_1_actuator_1
- added link arm_1_actuator_1a
- added link arm_1_actuator_1b; visual mesh filename=package://mearm_model/meshes/arm_1_right.stl scale=0.001 0.001 0.001
Joints:
- removed joint joint_2_mimic_0
- added joint joint_2_mimic_0a: type revolute, parent arm_1_actuator_0, child arm_1_actuator_1a, origin xyz=0.035 0 0, axis 0 0 1, limit lower=-1.57 upper=0.4 effort=1000.0 velocity=0.5, mimic joint=joint_2 multiplier=-1 offset=1.57
- added joint joint_2_mimic_0b: type revolute, parent arm_1_actuator_1a, child arm_1_actuator_1b, origin xyz=0 0 0, axis 0 0 1, limit lower=-1.57 upper=0.4 effort=1000.0 velocity=0.5, mimic joint=joint_1 multiplier=-1 offset=0

Commit message: added virtual link to mimic multiple joints in arm1 base

File: urdf/robot.urdf (robot description, URDF)
Before this commit: robot mearm, 11 links, 10 joints
Links:
- removed link arm_1
- added link arm_1a
- added link arm_1b; visual mesh filename=package://mearm_model/meshes/arm_1_left.stl scale=0.001 0.001 0.001; visual mesh filename=package://mearm_model/meshes/arm_1_right.stl scale=0.001 0.001 0.001
Joints:
- added joint arm1_mimic_0: type revolute, parent arm_1a, child arm_1b, origin xyz=0 0 0, axis 0 0 1, limit lower=-1.57 upper=0.4 effort=1000.0 velocity=0.5, mimic joint=joint_1 multiplier=-1 offset=0
- joint joint_2_mimic_1: child arm_1 -> arm_1a

Commit message: urdf code cleanup

File: urdf/robot.urdf (robot description, URDF)
Before this commit: robot mearm, 12 links, 11 joints
Links:
- removed link arm_0_1_connector
- removed link arm_1_actuator_0
- removed link arm_1_actuator_1a
- removed link arm_1_actuator_1b
- removed link arm_1_support
- added link arm_1_support_0; visual mesh filename=package://mearm_model/meshes/servo_actuator.stl scale=0.001 0.001 0.001
- added link arm_1_support_1a
- added link arm_1_support_1b; visual mesh filename=package://mearm_model/meshes/arm_1_right.stl scale=0.001 0.001 0.001
- added link connector; visual mesh filename=package://mearm_model/meshes/arm_1_connector.stl scale=0.001 0.001 0.001
- added link gripper_support; visual mesh filename=package://mearm_model/meshes/arm_1_right.stl scale=0.001 0.001 0.001
Joints:
- removed joint arm_1_support_mimic
- added joint gripper_support_mimic: type revolute, parent connector, child gripper_support, origin xyz=0.012 0.018 0.014 rpy=0 0 1.57, axis 0 0 1, limit lower=-1.57 upper=0.4 effort=1000.0 velocity=0.5, mimic joint=joint_2 multiplier=-1 offset=-1.57
- joint arm_0_connector_mimic: child arm_0_1_connector -> connector
- joint joint_2: child arm_1_actuator_0 -> arm_1_support_0
- joint joint_2_mimic_0a: child arm_1_actuator_1a -> arm_1_support_1a; parent arm_1_actuator_0 -> arm_1_support_0
- joint joint_2_mimic_0b: child arm_1_actuator_1b -> arm_1_support_1b; parent arm_1_actuator_1a -> arm_1_support_1a

Commit message: added base for gripper

File: urdf/robot.urdf (robot description, URDF)
Before this commit: robot mearm, 12 links, 11 joints
Links:
- added link gripper; visual mesh filename=package://mearm_model/meshes/gripper_base.stl scale=0.001 0.001 0.001
Joints:
- added joint gripper_holder: type revolute, parent arm_1b, child gripper, origin xyz=0.081 0.001 0.0 rpy=0 0 1.57, axis 0 0 1, limit lower=-1.57 upper=0.4 effort=1000.0 velocity=0.5, mimic joint=joint_2 multiplier=1 offset=-1.57

Commit message: added gripper

File: urdf/robot.urdf (robot description, URDF)
Before this commit: robot mearm, 13 links, 12 joints
Links:
- added link gripper_left; visual mesh filename=package://mearm_model/meshes/gripper_left.stl scale=0.001 0.001 0.001
- added link gripper_right; visual mesh filename=package://mearm_model/meshes/gripper_right.stl scale=0.001 0.001 0.001
- added link tool
- link gripper: geometry visual box size=0.024 0.018 0.012; visual mesh filename=package://mearm_model/meshes/gripper_base.stl scale=0.001 0.001 0.001
Joints:
- added joint joint_3: type revolute, parent gripper, child gripper_left, origin xyz=0.028 -0.003 -0.007 rpy=-1.57 0 0, axis 0 0 1, limit lower=0 upper=1.57 effort=1000.0 velocity=0.5
- added joint joint_3_mimic: type revolute, parent gripper, child gripper_right, origin xyz=0.028 -0.003 0.011 rpy=-1.57 0 0, axis 0 0 1, limit lower=0 upper=1.57 effort=1000.0 velocity=0.5, mimic joint=joint_3 multiplier=-1 offset=0
- added joint tool_joint: type fixed, parent gripper, child tool, origin xyz=0.043 -0.005 0.003 rpy=-1.57 0 0, axis 0 0 1

Commit message: added collision model

File: urdf/robot.urdf (robot description, URDF)
Before this commit: robot mearm, 16 links, 15 joints
Links:
- link arm_0_support: geometry collision mesh filename=package://mearm_model/meshes/arm_1_right.stl scale=0.001 0.001 0.001; visual mesh filename=package://mearm_model/meshes/arm_1_right.stl scale=0.001 0.001 0.001
- link arm_1_support_0: geometry collision mesh filename=package://mearm_model/meshes/servo_actuator.stl scale=0.001 0.001 0.001; visual mesh filename=package://mearm_model/meshes/servo_actuator.stl scale=0.001 0.001 0.001
- link arm_1_support_1b: geometry collision mesh filename=package://mearm_model/meshes/arm_1_right.stl scale=0.001 0.001 0.001; visual mesh filename=package://mearm_model/meshes/arm_1_right.stl scale=0.001 0.001 0.001
- link arm_1b: geometry collision mesh filename=package://mearm_model/meshes/arm_1_left.stl scale=0.001 0.001 0.001; collision mesh filename=package://mearm_model/meshes/arm_1_right.stl scale=0.001 0.001 0.001
- link connector: geometry collision mesh filename=package://mearm_model/meshes/arm_1_connector.stl scale=0.001 0.001 0.001; visual mesh filename=package://mearm_model/meshes/arm_1_connector.stl scale=0.001 0.001 0.001
- link gripper: geometry collision box size=0.024 0.018 0.012; collision mesh filename=package://mearm_model/meshes/gripper_base.stl scale=0.001 0.001 0.001
- link gripper_left: geometry collision mesh filename=package://mearm_model/meshes/gripper_left.stl scale=0.001 0.001 0.001; visual mesh filename=package://mearm_model/meshes/gripper_left.stl scale=0.001 0.001 0.001
- link gripper_right: geometry collision mesh filename=package://mearm_model/meshes/gripper_right.stl scale=0.001 0.001 0.001; visual mesh filename=package://mearm_model/meshes/gripper_right.stl scale=0.001 0.001 0.001
- link gripper_support: geometry collision mesh filename=package://mearm_model/meshes/arm_1_right.stl scale=0.001 0.001 0.001; visual mesh filename=package://mearm_model/meshes/arm_1_right.stl scale=0.001 0.001 0.001
